Commit message: setup_changes

File: install/robot_arm_moveit_config/share/robot_arm_moveit_config/config/robot_arm.ros2_control.xacro (robot description, xacro)
@@ -1,33 +1 @@
-<?xml version="1.0"?>
-<robot xmlns:xacro="http://www.ros.org/wiki/xacro">
-    <xacro:macro name="robot_arm_ros2_control" params="name initial_positions_file">
-        <xacro:property name="initial_positions" value="${xacro.load_yaml(initial_positions_file)['initial_positions']}"/>
-        <ros2_control name="${name}" type="system">
-            <hardware>
-                <!-- Simulation only. Replace with the STM32 hardware interface for the real arm. -->
-                <plugin>mock_components/GenericSystem</plugin>
-            </hardware>
-            <joint name="base_joint">
-                <command_interface name="position"/>
-                <state_interface name="position">
-                    <param name="initial_value">${initial_positions['base_joint']}</param>
-                </state_interface>
-                <state_interface name="velocity"/>
-            </joint>
-            <joint name="shoulder_joint">
-                <command_interface name="position"/>
-                <state_interface name="position">
-                    <param name="initial_value">${initial_positions['shoulder_joint']}</param>
-                </state_interface>
-                <state_interface name="velocity"/>
-            </joint>
-            <joint name="elbow_joint">
-                <command_interface name="position"/>
-                <state_interface name="position">
-                    <param name="initial_value">${initial_positions['elbow_joint']}</param>
-                </state_interface>
-                <state_interface name="velocity"/>
-            </joint>
-        </ros2_control>
-    </xacro:macro>
-</robot>
+/home/saicharan/autonomous_arm_ws/src/robot_arm_moveit_config/config/robot_arm.ros2_control.xacro

File: install/robot_arm_moveit_config/share/robot_arm_moveit_config/config/robot_arm.urdf.xacro (robot description, xacro)
@@ -1,9 +1 @@
-<?xml version="1.0"?>
-<robot xmlns:xacro="http://www.ros.org/wiki/xacro" name="robot_arm">
-    <xacro:arg name="initial_positions_file" default="initial_positions.yaml"/>
-    <!-- Robot description from the robot_arm package (geometry unchanged from CAD) -->
-    <xacro:include filename="$(find robot_arm)/description/urdf/robot_arm.urdf"/>
-    <!-- ros2_control (mock hardware for MoveIt testing) -->
-    <xacro:include filename="robot_arm.ros2_control.xacro"/>
-    <xacro:robot_arm_ros2_control name="MockSystem" initial_positions_file="$(arg initial_positions_file)"/>
-</robot>
+/home/saicharan/autonomous_arm_ws/src/robot_arm_moveit_config/config/robot_arm.urdf.xacro
