Commit message: URDF + MoveIt: joint limits for 300 / 500 mm actuators
- robot_arm.urdf: shoulder upper -0.022426 rad (-1.285 deg), elbow -0.149650 .. 1.007196 rad
  (-8.574 .. 57.708 deg); shoulder velocity 0.0420 rad/s, effort 166.6 (largest lever arm 166.6 mm)
- MoveIt joint_limits.yaml: shoulder max_velocity 0.0420 to match the URDF
- Start pose, saved poses and self-collision matrix re-checked: all still valid, no change needed
- URDF_CHANGES.md updated

Co-Authored-By: Claude Opus 5.5 <noreply@anthropic.com>
Claude-Session: https://claude.ai/code/session_01CJ3NfDdD4QrzaejrXgfX5S

File: src/robot_arm/description/urdf/robot_arm.urdf (robot description, URDF)
Before this commit: robot robot_arm, 18 links, 17 joints
Joints:
- joint elbow_joint: limit lower=-0.189703 upper=0.981815 effort=197.4 velocity=0.0355 -> lower=-0.149650 upper=1.007196 effort=197.4 velocity=0.0355
- joint shoulder_joint: limit lower=-1.570796 upper=-0.052638 effort=164.4 velocity=0.0426 -> lower=-1.570796 upper=-0.022426 effort=166.6 velocity=0.0420
